Commit message: configured urdf file

File: src/bumperbot_description/urdf/bumperbot.urdf (robot description, URDF)
Before this commit: robot bumperbot, 2 links, 0 joints
Links:
- added link caster_front_link; visual mesh filename=package://bumperbot_description/meshes/caster_front_link.STL
- added link caster_rear_link; visual mesh filename=package://bumperbot_description/meshes/caster_rear_link.STL
- added link wheel_left_link; visual mesh filename=package://bumperbot_description/meshes/wheel_left_link.STL
- added link wheel_right_link; visual mesh filename=package://bumperbot_description/meshes/wheel_right_link.STL
Joints:
- added joint base_joint: type fixed, parent base_footprint, child base_link, origin xyz=0 0 0.033 rpy=0 0 0
- added joint caster_front_joint: type fixed, parent base_link, child caster_front_link, origin xyz=0.0475 0 -0.0275 rpy=0 0 0
- added joint caster_rear_joint: type fixed, parent base_link, child caster_rear_link, origin xyz=-0.0475 0 -0.0275 rpy=0 0 0
- added joint wheel_left_joint: type continuous, parent base_link, child wheel_left_link, origin xyz=0 0.07 0 rpy=0 0 0, axis 0 1 0
- added joint wheel_right_joint: type continuous, parent base_link, child wheel_right_link, origin xyz=0 -0.07 0 rpy=0 0 0, axis 0 1 0
