Commit message: added ROS control in bumperbot_gazebo.xacro

File: src/bumperbot_description/urdf/bumperbot_gazebo.xacro (robot description, xacro)
@@ -1,4 +1,24 @@
 <?xml version="1.0"?>
 <robot name="bumperbot" xmlns:xacro="http://ros.org/wiki/xacro">
+    <transmission name="wheel_right_transmission">
+        <type>transmission_interface/SimpleTransmission</type>
+        <joint name="wheel_right_joint">
+            <hardwareInterface>hardware_interface/VelocityJointInterface</hardwareInterface>
+        </joint>
+        <actuator name="wheel_right_motor">
+            <hardwareInterface>hardware_interface/VelocityJointInterface</hardwareInterface>
+            <mechanicalReduction>1.0</mechanicalReduction>
+        </actuator>
+    </transmission>
+    <transmission name="wheel_left_transmission">
+        <type>transmission_interface/SimpleTransmission</type>
+        <joint name="wheel_left_joint">
+            <hardwareInterface>hardware_interface/VelocityJointInterface</hardwareInterface>
+        </joint>
+        <actuator name="wheel_left_motor">
+            <hardwareInterface>hardware_interface/VelocityJointInterface</hardwareInterface>
+            <mechanicalReduction>1.0</mechanicalReduction>
+        </actuator>
+    </transmission>
     <gazebo reference="wheel_right_link">
         <mu1>100000000000000.0</mu1>
@@ -37,3 +57,9 @@
         <fdir>1 0 0</fdir>
     </gazebo>
+    <gazebo>
+        <plugin name="gazebo_ros_control" filename="libgazebo_ros_control.so">
+            <robotSimType>gazebo_ros_control/DefaultRobotHwSim</robotSimType>
+            <legacyModeNS>true</legacyModeNS>
+        </plugin>
+    </gazebo>
 </robot>
